Commit message: ✨ added hand wrist for all robotic hand

File: src/fourier_robot_descriptions/assets/urdf/fourier_left_hand_12dof.urdf (robot description, URDF)
Before this commit: robot fourier_left_hand_12dof, 18 links, 17 joints
Links:
- added link L_hand_wrist_link
Joints:
- added joint L_hand_wrist_joint: type fixed, parent L_hand_base_link, child L_hand_wrist_link, origin xyz=0 0 0 rpy=0 0 0, axis 0 0 0

File: src/fourier_robot_descriptions/assets/urdf/fourier_left_hand_6dof.urdf (robot description, URDF)
Before this commit: robot fourier_left_hand_6dof, 17 links, 16 joints
Links:
- added link L_hand_wrist_link
Joints:
- added joint L_hand_wrist_joint: type fixed, parent L_hand_base_link, child L_hand_wrist_link, origin xyz=0 0 0 rpy=-0.0872 0 0, axis 0 0 0

File: src/fourier_robot_descriptions/assets/urdf/fourier_right_hand_12dof.urdf (robot description, URDF)
Before this commit: robot fourier_right_hand_12dof, 18 links, 17 joints
Links:
- added link R_hand_wrist_link
Joints:
- added joint R_hand_wrist_joint: type fixed, parent R_hand_base_link, child R_hand_wrist_link, origin xyz=0 0 0 rpy=0 0 0, axis 0 0 0

File: src/fourier_robot_descriptions/assets/urdf/fourier_right_hand_6dof.urdf (robot description, URDF)
Before this commit: robot fourier_right_hand_6dof, 17 links, 16 joints
Links:
- added link R_hand_wrist_link
Joints:
- added joint R_hand_wrist_joint: type fixed, parent R_hand_base_link, child R_hand_wrist_link, origin xyz=0 0 0 rpy=0.0872 0 0, axis 0 0 0

File: src/fourier_robot_descriptions/assets/urdf/gr1t1_fourier_hand_12dof.urdf (robot description, URDF)
Before this commit: robot GR1T1_fourier_hand_12dof, 73 links, 72 joints
Links:
- added link L_hand_wrist_link
- added link R_hand_wrist_link
Joints:
- added joint L_hand_wrist_joint: type fixed, parent L_hand_base_link, child L_hand_wrist_link, origin xyz=0 0 0 rpy=0 0 0, axis 0 0 0
- added joint R_hand_wrist_joint: type fixed, parent R_hand_base_link, child R_hand_wrist_link, origin xyz=0 0 0 rpy=0 0 0, axis 0 0 0

File: src/fourier_robot_descriptions/assets/urdf/gr1t1_fourier_hand_12dof_v2.urdf (robot description, URDF)
Before this commit: robot GR1T1_fourier_hand_12dof_v2, 73 links, 72 joints
Links:
- added link L_hand_wrist_link
- added link R_hand_wrist_link
Joints:
- added joint L_hand_wrist_joint: type fixed, parent L_hand_base_link, child L_hand_wrist_link, origin xyz=0 0 0 rpy=0 0 0, axis 0 0 0
- added joint R_hand_wrist_joint: type fixed, parent R_hand_base_link, child R_hand_wrist_link, origin xyz=0 0 0 rpy=0 0 0, axis 0 0 0

File: src/fourier_robot_descriptions/assets/urdf/gr1t1_fourier_hand_6dof.urdf (robot description, URDF)
Before this commit: robot GR1T1_fourier_hand_6dof, 71 links, 70 joints
Links:
- added link L_hand_wrist_link
- added link R_hand_wrist_link
Joints:
- added joint L_hand_wrist_joint: type fixed, parent L_hand_base_link, child L_hand_wrist_link, origin xyz=0 0 0 rpy=-0.0872 0 0, axis 0 0 0
- added joint R_hand_wrist_joint: type fixed, parent R_hand_base_link, child R_hand_wrist_link, origin xyz=0 0 0 rpy=0.0872 0 0, axis 0 0 0

File: src/fourier_robot_descriptions/assets/urdf/gr1t1_inspire_hand.urdf (robot description, URDF)
Before this commit: robot GR1T1_inspire_hand, 73 links, 72 joints
Links:
- added link L_hand_wrist_link
- added link R_hand_wrist_link
Joints:
- added joint L_hand_wrist_joint: type fixed, parent L_hand_base_link, child L_hand_wrist_link, origin xyz=0 0 0 rpy=0 0 0, axis 0 0 0
- added joint R_hand_wrist_joint: type fixed, parent R_hand_base_link, child R_hand_wrist_link, origin xyz=0 0 0 rpy=0 0 0, axis 0 0 0

File: src/fourier_robot_descriptions/assets/urdf/gr1t2_fourier_hand_12dof.urdf (robot description, URDF)
Before this commit: robot GR1T2_fourier_hand_12dof, 73 links, 72 joints
Links:
- added link L_hand_wrist_link
- added link R_hand_wrist_link
Joints:
- added joint L_hand_wrist_joint: type fixed, parent L_hand_base_link, child L_hand_wrist_link, origin xyz=0 0 0 rpy=0 0 0, axis 0 0 0
- added joint R_hand_wrist_joint: type fixed, parent R_hand_base_link, child R_hand_wrist_link, origin xyz=0 0 0 rpy=0 0 0, axis 0 0 0

File: src/fourier_robot_descriptions/assets/urdf/gr1t2_fourier_hand_6dof.urdf (robot description, URDF)
Before this commit: robot GR1T2_fourier_hand_6dof, 71 links, 70 joints
Links:
- added link L_hand_wrist_link
- added link R_hand_wrist_link
Joints:
- added joint L_hand_wrist_joint: type fixed, parent L_hand_base_link, child L_hand_wrist_link, origin xyz=0 0 0 rpy=-0.0872 0 0, axis 0 0 0
- added joint R_hand_wrist_joint: type fixed, parent R_hand_base_link, child R_hand_wrist_link, origin xyz=0 0 0 rpy=0.0872 0 0, axis 0 0 0

File: src/fourier_robot_descriptions/assets/urdf/gr1t2_inspire_hand.urdf (robot description, URDF)
Before this commit: robot GR1T2_inspire_hand, 73 links, 72 joints
Links:
- added link L_hand_wrist_link
- added link R_hand_wrist_link
Joints:
- added joint L_hand_wrist_joint: type fixed, parent L_hand_base_link, child L_hand_wrist_link, origin xyz=0 0 0 rpy=0 0 0, axis 0 0 0
- added joint R_hand_wrist_joint: type fixed, parent R_hand_base_link, child R_hand_wrist_link, origin xyz=0 0 0 rpy=0 0 0, axis 0 0 0

File: src/fourier_robot_descriptions/assets/urdf/gr2t2_fourier_hand_12dof.urdf (robot description, URDF)
Before this commit: robot GR2T2_fourier_hand_12dof, 71 links, 70 joints
Links:
- added link L_hand_wrist_link
- added link R_hand_wrist_link
Joints:
- added joint L_hand_wrist_joint: type fixed, parent L_hand_base_link, child L_hand_wrist_link, origin xyz=0 0 0 rpy=0 0 0, axis 0 0 0
- added joint R_hand_wrist_joint: type fixed, parent R_hand_base_link, child R_hand_wrist_link, origin xyz=0 0 0 rpy=0 0 0, axis 0 0 0

File: src/fourier_robot_descriptions/assets/urdf/gr2t2_fourier_hand_6dof.urdf (robot description, URDF)
Before this commit: robot GR2T2_fourier_hand_6dof, 69 links, 68 joints
Links:
- added link L_hand_wrist_link
- added link R_hand_wrist_link
Joints:
- added joint L_hand_wrist_joint: type fixed, parent L_hand_base_link, child L_hand_wrist_link, origin xyz=0 0 0 rpy=-0.0872 0 0, axis 0 0 0
- added joint R_hand_wrist_joint: type fixed, parent R_hand_base_link, child R_hand_wrist_link, origin xyz=0 0 0 rpy=0.0872 0 0, axis 0 0 0

File: src/fourier_robot_descriptions/assets/urdf/gr2t2d_fourier_hand_6dof.urdf (robot description, URDF)
Before this commit: robot GR2T2v2_fourier_hand_6dof, 69 links, 68 joints
Links:
- added link L_hand_wrist_link
- added link R_hand_wrist_link
Joints:
- added joint L_hand_wrist_joint: type fixed, parent L_hand_base_link, child L_hand_wrist_link, origin xyz=0 0 0 rpy=-0.0872 0 0, axis 0 0 0
- added joint R_hand_wrist_joint: type fixed, parent R_hand_base_link, child R_hand_wrist_link, origin xyz=0 0 0 rpy=0.0872 0 0, axis 0 0 0

File: src/fourier_robot_descriptions/assets/urdf/gr2t2v2_fourier_hand_12dof.urdf (robot description, URDF)
Before this commit: robot GR2T2v2_fourier_hand_12dof, 71 links, 70 joints
Links:
- added link L_hand_wrist_link
- added link R_hand_wrist_link
Joints:
- added joint L_hand_wrist_joint: type fixed, parent L_hand_base_link, child L_hand_wrist_link, origin xyz=0 0 0 rpy=0 0 0, axis 0 0 0
- added joint R_hand_wrist_joint: type fixed, parent R_hand_base_link, child R_hand_wrist_link, origin xyz=0 0 0 rpy=0 0 0, axis 0 0 0

File: src/fourier_robot_descriptions/assets/urdf/gr2t2v2_fourier_hand_6dof.urdf (robot description, URDF)
Before this commit: robot GR2T2v2_fourier_hand_6dof, 69 links, 68 joints
Links:
- added link L_hand_wrist_link
- added link R_hand_wrist_link
Joints:
- added joint L_hand_wrist_joint: type fixed, parent L_hand_base_link, child L_hand_wrist_link, origin xyz=0 0 0 rpy=-0.0872 0 0, axis 0 0 0
- added joint R_hand_wrist_joint: type fixed, parent R_hand_base_link, child R_hand_wrist_link, origin xyz=0 0 0 rpy=0.0872 0 0, axis 0 0 0

File: src/fourier_robot_descriptions/assets/urdf/inspire_left_hand.urdf (robot description, URDF)
Before this commit: robot inspire_left_hand, 18 links, 17 joints
Links:
- added link L_hand_wrist_link
Joints:
- added joint L_hand_wrist_joint: type fixed, parent L_hand_base_link, child L_hand_wrist_link, origin xyz=0 0 0 rpy=0 0 0, axis 0 0 0

File: src/fourier_robot_descriptions/assets/urdf/inspire_right_hand.urdf (robot description, URDF)
Before this commit: robot inspire_right_hand, 18 links, 17 joints
Links:
- added link R_hand_wrist_link
Joints:
- added joint R_hand_wrist_joint: type fixed, parent R_hand_base_link, child R_hand_wrist_link, origin xyz=0 0 0 rpy=0 0 0, axis 0 0 0

File: src/fourier_robot_descriptions/assets/urdf/qinglong_fourier_hand_6dof.urdf (robot description, URDF)
Before this commit: robot openloong_fourier_hand_6dof, 70 links, 69 joints
Links:
- added link L_hand_wrist_link
- added link R_hand_wrist_link
Joints:
- added joint L_hand_wrist_joint: type fixed, parent L_hand_base_link, child L_hand_wrist_link, origin xyz=0 0 0 rpy=-0.0872 0 0, axis 0 0 0
- added joint R_hand_wrist_joint: type fixed, parent R_hand_base_link, child R_hand_wrist_link, origin xyz=0 0 0 rpy=0.0872 0 0, axis 0 0 0
