Commit message: 🎨 Updating the urdf name and folder structure

File: src/fourier_robot_descriptions/assets/base_urdf/fourier_left_hand_12dof.urdf (robot description, URDF)
Before this commit: robot fourier_left_hand_6dof, 18 links, 17 joints
Links:
- added link L_index_metacarpal_link, mass 0.028947; collision mesh filename=../meshes/fourier_hand_12dof_v2/L_index_metacarpal_link.STL; visual mesh filename=../meshes/fourier_hand_12dof_v2/L_index_metacarpal_link.STL
- link L_hand_base_link: mass 0.29928 -> 0.26434; geometry collision mesh filename=../meshes/fourier_hand_12dof_v2/L_hand_base_link.STL; visual mesh filename=../meshes/fourier_hand_12dof_v2/L_hand_base_link.STL
- link L_index_intermediate_link: mass 0.0027085 -> 0.019358; geometry collision mesh filename=../meshes/fourier_hand_12dof_v2/L_index_intermediate_link.S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; visual mesh filename=../meshes/fourier_hand_12dof_v2/L_index_intermediate_link.S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
- link L_index_proximal_link: mass 0.01124444 -> 0.035619; geometry collision mesh filename=../meshes/fourier_hand_12dof_v2/L_index_proximal_link.STL; visual mesh filename=../meshes/fourier_hand_12dof_v2/L_index_proximal_link.STL
- link L_middle_intermediate_link: mass 0.0032739 -> 0.022377; geometry collision mesh filename=../meshes/fourier_hand_12dof_v2/L_middle_intermediate_link.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; visual mesh filename=../meshes/fourier_hand_12dof_v2/L_middle_intermediate_link.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
- link L_middle_proximal_link: mass 0.01124444 -> 0.035619; geometry collision mesh filename=../meshes/fourier_hand_12dof_v2/L_middle_proximal_link.STL; visual mesh filename=../meshes/fourier_hand_12dof_v2/L_middle_proximal_link.STL
- link L_pinky_intermediate_link: mass 0.0024076 -> 0.01622; geometry collision mesh filename=../meshes/fourier_hand_12dof_v2/L_pinky_intermediate_link.S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; visual mesh filename=../meshes/fourier_hand_12dof_v2/L_pinky_intermediate_link.S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
- link L_pinky_proximal_link: mass 0.01124444 -> 0.035619; geometry collision mesh filename=../meshes/fourier_hand_12dof_v2/L_pinky_proximal_link.STL; visual mesh filename=../meshes/fourier_hand_12dof_v2/L_pinky_proximal_link.STL
- link L_ring_intermediate_link: mass 0.0027085 -> 0.019358; geometry collision mesh filename=../meshes/fourier_hand_12dof_v2/L_ring_intermediate_link.STL; visual mesh filename=../meshes/fourier_hand_12dof_v2/L_ring_intermediate_link.STL
- link L_ring_proximal_link: mass 0.01124444 -> 0.035619; geometry collision mesh filename=../meshes/fourier_hand_12dof_v2/L_ring_proximal_link.STL; visual mesh filename=../meshes/fourier_hand_12dof_v2/L_ring_proximal_link.STL
- link L_thumb_distal_link: mass 0.018024 -> 0.021803; geometry collision mesh filename=../meshes/fourier_hand_12dof_v2/L_thumb_distal_link.STL; visual mesh filename=../meshes/fourier_hand_12dof_v2/L_thumb_distal_link.STL
- link L_thumb_proximal_pitch_link: mass 0.060766 -> 0.047552; geometry collision mesh filename=../meshes/fourier_hand_12dof_v2/L_thumb_proximal_pitch_link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; visual mesh filename=../meshes/fourier_hand_12dof_v2/L_thumb_proximal_pitch_link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
- link L_thumb_proximal_yaw_link: mass 0.0084328 -> 0.034977; geometry collision mesh filename=../meshes/fourier_hand_12dof_v2/L_thumb_proximal_yaw_link.S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; visual mesh filename=../meshes/fourier_hand_12dof_v2/L_thumb_proximal_yaw_link.S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
Joints:
- added joint L_index_metacarpal_joint: type revolute, parent L_hand_base_link, child L_index_metacarpal_link, origin xyz=0.0305 -0.0113 -0.088496 rpy=0 1.5295 -3.1416, axis 0 1 0, limit lower=0 upper=0.295 effort=0 velocity=0
- joint L_hand_wrist_joint: origin xyz=0 0 0 rpy=-0.0872 0 0 -> xyz=0 0 0 rpy=0 0 0
- joint L_index_intermediate_joint: limit lower=-1.791 upper=0 effort=0 velocity=0 -> lower=-1.4835 upper=0 effort=0 velocity=0; mimic joint=L_index_proximal_joint multiplier=0.975 offset=0 -> (none); origin xyz=0.031533 -0.0054444 0 rpy=0 0.00014037 -0.0018338 -> xyz=0.038938 0.0021905 0 rpy=0 0 -0.040106
- joint L_index_proximal_joint: limit lower=-1.592 upper=0 effort=0 velocity=0 -> lower=-1.4172 upper=0 effort=0 velocity=0; origin xyz=0.026868 -0.0123 -0.093989 rpy=0 1.5184 0 -> xyz=0.012 0 0 rpy=-3.1416 0 0.041438; parent L_hand_base_link -> L_index_metacarpal_link
- joint L_index_tip_joint: origin xyz=0.0390 -0.0020 0 rpy=0 0 0 -> xyz=0.047 -0.003 0 rpy=0 0 0
- joint L_middle_intermediate_joint: limit lower=-1.792 upper=0 effort=0 velocity=0 -> lower=-1.4835 upper=0 effort=0 velocity=0; mimic joint=L_middle_proximal_joint multiplier=0.975 offset=0 -> (none); origin xyz=0.031521 -0.0055139 0 rpy=0 0.00015517 0.0048744 -> xyz=0.038912 0.0026251 0 rpy=0 -7.4325E-05 -0.04236
- joint L_middle_proximal_joint: limit lower=-1.593 upper=0 effort=0 velocity=0 -> lower=-1.4172 upper=0 effort=0 velocity=0; origin xyz=0.0085 -0.0123 -0.095992 rpy=0 1.5708 0 -> xyz=0.0091 -0.0113 -0.10005 rpy=-1.5685 1.5182 -1.5685
- joint L_middle_tip_joint: origin xyz=0.047 -0.0025 0 rpy=0 0 0 -> xyz=0.055 -0.003 0 rpy=0 0 0
- joint L_pinky_intermediate_joint: limit lower=-1.791 upper=0 effort=0 velocity=0 -> lower=-1.4835 upper=0 effort=0 velocity=0; mimic joint=L_pinky_proximal_joint multiplier=0.975 offset=0 -> (none); origin xyz=0.031532 -0.005451 0 rpy=0 0.00032164 -0.011403 -> xyz=0.038963 0.0016981 0 rpy=0 0 -0.036802
- joint L_pinky_proximal_joint: limit lower=-1.592 upper=0 effort=0 velocity=0 -> lower=-1.4172 upper=0 effort=0 velocity=0; origin xyz=-0.028228 -0.0123 -0.094012 rpy=3.1416 1.4661 3.1416 -> xyz=-0.031472 -0.0113 -0.099245 rpy=-2.8742 1.4622 -2.8727
- joint L_pinky_tip_joint: origin xyz=0.033 -0.0015 0 rpy=0 0 0 -> xyz=0.038 -0.003 0 rpy=0 0 0
- joint L_ring_intermediate_joint: limit lower=-1.791 upper=0 effort=0 velocity=0 -> lower=-1.4835 upper=0 effort=0 velocity=0; mimic joint=L_ring_proximal_joint multiplier=0.975 offset=0 -> (none); origin xyz=0.031531 -0.0054567 0.00025 rpy=0 0.00014037 -0.0025338 -> xyz=0.038938 0.0021905 0 rpy=0 0 -0.040106
- joint L_ring_proximal_joint: limit lower=-1.593 upper=0 effort=0 velocity=0 -> lower=-1.4172 upper=0 effort=0 velocity=0; origin xyz=-0.010211 -0.0123 -0.095924 rpy=3.1416 1.5184 3.1416 -> xyz=-0.011187 -0.0113 -0.10003 rpy=-2.4727 1.504 -2.4716
- joint L_ring_tip_joint: origin xyz=0.0385 -0.0015 0 rpy=0 0 0 -> xyz=0.045 -0.003 0 rpy=0 0 0
- joint L_thumb_distal_joint: limit lower=0 upper=1.248 effort=0 velocity=0 -> lower=0 upper=1.2078 effort=0 velocity=0; mimic joint=L_thumb_proximal_pitch_joint multiplier=1.06 offset=0 -> (none); origin xyz=0.061549 0.007464 0 rpy=0 1.7448E-05 -0.055652 -> xyz=0.051711 0.0054792 0 rpy=0 0 -0.12355
- joint L_thumb_proximal_pitch_joint: limit lower=0 upper=1.143 effort=0 velocity=0 -> lower=0 upper=1.206 effort=0 velocity=0; origin xyz=0.021749 -0.00016321 0 rpy=-1.5708 0 -0.0052052 -> xyz=0.03385 -0.0078588 -0.0005 rpy=-1.5708 0.037538 -0.22813
- joint L_thumb_proximal_yaw_joint: limit lower=-1.696 upper=0 effort=0 velocity=0 -> lower=-1.3579 upper=0 effort=0 velocity=0; origin xyz=0.022 -0.0155 -0.022992 rpy=0 0 0 -> xyz=0.014 -0.012 -0.022446 rpy=0 0 0
- joint L_thumb_tip_joint: origin xyz=0.0305 -0.001 0 rpy=0 0 0 -> xyz=0.035 0.001 0 rpy=0 0 0
